File: PR9010.sch (EAGLE design)
At the start: 60 parts, among them J1 AVR_SPI_PRG_6NS, U1 SI4703, U2 Tiny85-20-SMT, Y1 32.768kHz

Commit message: fixed prefixes
Parts:
- C1, C10, C13, C2, C6, C8: value (none) -> 1.0uF
- C14: value 4.7uF -> 1.0uF
Changed lines of the file:
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@@
 <?xml version="1.0" encoding="utf-8"?>
 <!DOCTYPE eagle SYSTEM "eagle.dtd">
-<eagle version="6.6.0">
+<eagle version="7.2.0">
 <drawing>
 <settings>
@@
 <part name="R5" library="resistor" deviceset="R-US_" device="R0603" value="1K"/>
 <part name="GND25" library="SparkFun-Aesthetics" deviceset="GND" device=""/>
-<part name="C8" library="SparkFun-Capacitors" deviceset="1.0UF-25V-+80/-20(0805)" device=""/>
+<part name="C8" library="SparkFun-Capacitors" deviceset="1.0UF-25V-+80/-20(0805)" device="" value="1.0uF"/>
 <part name="L1" library="SparkFun-Passives" deviceset="INDUCTOR" device="0805"/>
-<part name="C10" library="SparkFun-Capacitors" deviceset="1.0UF-25V-+80/-20(0805)" device=""/>
+<part name="C10" library="SparkFun-Capacitors" deviceset="1.0UF-25V-+80/-20(0805)" device="" value="1.0uF"/>
 <part name="GND26" library="SparkFun" deviceset="GND" device=""/>
-<part name="C13" library="SparkFun-Capacitors" deviceset="1.0UF-25V-+80/-20(0805)" device=""/>
-<part name="C1" library="SparkFun-Capacitors" deviceset="1.0UF-25V-+80/-20(0805)" device=""/>
-<part name="C2" library="SparkFun-Capacitors" deviceset="1.0UF-25V-+80/-20(0805)" device=""/>
-<part name="C6" library="SparkFun-Capacitors" deviceset="1.0UF-25V-+80/-20(0805)" device=""/>
+<part name="C13" library="SparkFun-Capacitors" deviceset="1.0UF-25V-+80/-20(0805)" device="" value="1.0uF"/>
+<part name="C1" library="SparkFun-Capacitors" deviceset="1.0UF-25V-+80/-20(0805)" device="" value="1.0uF"/>
+<part name="C2" library="SparkFun-Capacitors" deviceset="1.0UF-25V-+80/-20(0805)" device="" value="1.0uF"/>
+<part name="C6" library="SparkFun-Capacitors" deviceset="1.0UF-25V-+80/-20(0805)" device="" value="1.0uF"/>
 <part name="GND27" library="SparkFun" deviceset="GND" device=""/>
 <part name="PWRIN" library="SparkFun-Connectors" deviceset="M02" device="PTH3"/>
-<part name="C14" library="SparkFun-Capacitors" deviceset="1.0UF-25V-+80/-20(0805)" device="" value="4.7uF"/>
+<part name="C14" library="SparkFun-Capacitors" deviceset="1.0UF-25V-+80/-20(0805)" device="" value="1.0uF"/>
 <part name="R6" library="SparkFun-Passives" deviceset="RESISTOR" device="0805-RES" value="4.7K"/>
 <part name="R13" library="SparkFun-Passives" deviceset="RESISTOR" device="0805-RES" value="4.7K"/>
@@
 <instance part="GND4" gate="1" x="27.94" y="15.24"/>
 <instance part="GND10" gate="1" x="-25.4" y="40.64"/>
-<instance part="P+3" gate="G$1" x="34.798" y="60.96"/>
-<instance part="P+4" gate="G$1" x="41.148" y="60.96"/>
-<instance part="P+5" gate="G$1" x="48.006" y="60.96"/>
-<instance part="P+6" gate="G$1" x="53.34" y="72.39"/>
-<instance part="P+18" gate="G$1" x="-22.86" y="73.66"/>
+<instance part="P+3" gate="1" x="34.798" y="60.96"/>
+<instance part="P+4" gate="1" x="41.148" y="60.96"/>
+<instance part="P+5" gate="1" x="48.006" y="60.96"/>
+<instance part="P+6" gate="1" x="53.34" y="72.39"/>
+<instance part="P+18" gate="1" x="-22.86" y="73.66"/>
 <instance part="FMIC_IO" gate="G$1" x="-38.1" y="66.04" smashed="yes">
 <attribute name="NAME" x="-38.1" y="74.93" size="1.778" layer="95"/>
@@
 <instance part="GND24" gate="1" x="-18.288" y="128.524"/>
 <instance part="U2" gate="G$1" x="176.276" y="124.46"/>
-<instance part="P+1" gate="G$1" x="155.956" y="132.08"/>
+<instance part="P+1" gate="1" x="155.956" y="132.08"/>
 <instance part="GND7" gate="1" x="155.956" y="116.84"/>
 <instance part="GND8" gate="1" x="139.7" y="127"/>
 <instance part="GND12" gate="1" x="129.54" y="127"/>
-<instance part="P+2" gate="G$1" x="129.54" y="137.16"/>
-<instance part="P+13" gate="G$1" x="139.7" y="137.16"/>
+<instance part="P+2" gate="1" x="129.54" y="137.16"/>
+<instance part="P+13" gate="1" x="139.7" y="137.16"/>
 <instance part="STA_CH" gate="G$1" x="200.152" y="108.204" smashed="yes" rot="R270">
 <attribute name="NAME" x="197.612" y="114.554" size="1.778" layer="95"/>
@@
 <instance part="LED1" gate="G$1" x="204.978" y="100.33"/>
 <instance part="GND14" gate="1" x="204.978" y="92.71"/>
-<instance part="P+9" gate="G$1" x="219.71" y="137.414"/>
+<instance part="P+9" gate="1" x="219.71" y="137.414"/>
 <instance part="GND16" gate="1" x="219.71" y="116.84"/>
 <instance part="R5" gate="G$1" x="198.628" y="102.87" smashed="yes" rot="R180">
@@
 <segment>
 <wire x1="34.798" y1="60.96" x2="34.798" y2="57.658" width="0.1524" layer="91"/>
-<pinref part="P+3" gate="G$1" pin="VCC"/>
+<pinref part="P+3" gate="1" pin="VCC"/>
 <pinref part="R13" gate="G$1" pin="2"/>
 </segment>
 <segment>
 <wire x1="41.148" y1="60.96" x2="41.148" y2="57.912" width="0.1524" layer="91"/>
-<pinref part="P+4" gate="G$1" pin="VCC"/>
+<pinref part="P+4" gate="1" pin="VCC"/>
 <pinref part="R6" gate="G$1" pin="2"/>
 </segment>
 <segment>
 <wire x1="48.006" y1="60.96" x2="48.006" y2="58.42" width="0.1524" layer="91"/>
-<pinref part="P+5" gate="G$1" pin="VCC"/>
+<pinref part="P+5" gate="1" pin="VCC"/>
 <pinref part="R14" gate="G$1" pin="2"/>
 </segment>
 <segment>
 <wire x1="-22.86" y1="63.5" x2="-22.86" y2="73.66" width="0.1524" layer="91"/>
-<pinref part="P+18" gate="G$1" pin="VCC"/>
+<pinref part="P+18" gate="1" pin="VCC"/>
 <wire x1="-22.86" y1="63.5" x2="-27.94" y2="63.5" width="0.1524" layer="91"/>
 <pinref part="FMIC_IO" gate="G$1" pin="7"/>
@@
 <segment>
 <pinref part="U2" gate="G$1" pin="VCC"/>
-<pinref part="P+1" gate="G$1" pin="VCC"/>
+<pinref part="P+1" gate="1" pin="VCC"/>
 <wire x1="161.036" y1="132.08" x2="155.956" y2="132.08" width="0.1524" layer="91"/>
 </segment>
 <segment>
 <pinref part="L3" gate="G$1" pin="1"/>
-<pinref part="P+6" gate="G$1" pin="VCC"/>
+<pinref part="P+6" gate="1" pin="VCC"/>
 <wire x1="53.34" y1="72.39" x2="53.34" y2="68.58" width="0.1524" layer="91"/>
 </segment>
@@
 <pinref part="J1" gate="G$1" pin="2"/>
 <wire x1="219.71" y1="137.414" x2="219.71" y2="129.54" width="0.1524" layer="91"/>
-<pinref part="P+9" gate="G$1" pin="VCC"/>
-</segment>
-<segment>
-<pinref part="P+2" gate="G$1" pin="VCC"/>
+<pinref part="P+9" gate="1" pin="VCC"/>
+</segment>
+<segment>
+<pinref part="P+2" gate="1" pin="VCC"/>
 <pinref part="C3" gate="G$1" pin="1"/>
 </segment>
 <segment>
-<pinref part="P+13" gate="G$1" pin="VCC"/>
+<pinref part="P+13" gate="1" pin="VCC"/>
 <pinref part="C4" gate="G$1" pin="1"/>
 </segment>

Commit message: Prefix changes
Prefix changes
Parts:
- removed AMP: TPA2005D1DGN, SparkFun-AnalogIC:TPA2005D1DGN
- removed ANT: M3_SCREW_POST, PR_Libraries:M3_SCREW_POST
- removed L4: 2.5 kOhm @ 100MHz, SparkFun-Passives:INDUCTOR0603
- removed U$5: RV170SF_TAIWANA_POT_SW, PR_Libraries:RV170SF_TAIWANA_POT_SW
- added J2: AVR_SPI_PRG_6NS, SparkFun-Connectors:AVR_SPI_PRG_6NS
- added L2: 2.5k@100MHz, SparkFun-Passives:INDUCTOR0603
- added R11: 40.2K, resistor:R-US_R0603
- added U3: Tiny85-20-SMT, SparkFun-DigitalIC:ATTINY45TINY85-20-SMT
- C1: value 1.0uF -> 220uF; device SparkFun-Capacitors:1.0UF-25V-+80/-20(0805) -> SparkFun-Passives:CAP_POLC
- C11, C9: value .033uf -> 1.0uF; device resistor:C-USC0603 -> SparkFun-Capacitors:1.0UF-25V-+80/-20(0805)
- C12: value 10uf -> .1uf
- C13: value 1.0uF -> .033uf; device SparkFun-Capacitors:1.0UF-25V-+80/-20(0805) -> resistor:C-USC0603
- C14: value 1.0uF -> 10uf; device SparkFun-Capacitors:1.0UF-25V-+80/-20(0805) -> SparkFun-Passives:CAP0805
- C15: value 22pf -> 10uf; device SparkFun-Passives:CAP0805 -> resistor:C-USC0603
- C16: value 100nF -> .033uf; device SparkFun-Passives:CAP0805 -> resistor:C-USC0603
- C17: value 100pf -> 1uf
- C18: device resistor:C-USC0603 -> SparkFun-Passives:CAP0805
- C19: value 220uF -> .1uf; device SparkFun-Passives:CAP_POLC -> SparkFun-Passives:CAP0805
- C20: value (none) -> 100pf
- C3: value .1uf -> 1.0uF; device SparkFun-Passives:CAP0805 -> SparkFun-Capacitors:1.0UF-25V-+80/-20(0805)
- C4: value 10uf -> 22pf
- C5: value 1uf -> 22pf
- C6: value 1.0uF -> (none); device SparkFun-Capacitors:1.0UF-25V-+80/-20(0805) -> SparkFun-Passives:CAP0805
- C7: value 22pf -> 1.0uF; device SparkFun-Passives:CAP0805 -> SparkFun-Capacitors:1.0UF-25V-+80/-20(0805)
- J1: value AVR_SPI_PRG_6NS -> M3_SCREW_POST; device SparkFun-Connectors:AVR_SPI_PRG_6NS -> PR_Libraries:M3_SCREW_POST
- L3: value 2.5k@100MHz -> 2.5 kOhm @ 100MHz
- R1: value (none) -> RV170SF_TAIWANA_POT_SW; device SparkFun-Passives:RESISTOR0805-RES -> PR_Libraries:RV170SF_TAIWANA_POT_SW
- R10: value 10K -> (none)
- R13: value 4.7K -> 40.2K; device SparkFun-Passives:RESISTOR0805-RES -> resistor:R-US_R0603
- R14: value 4.7K -> 1K; device SparkFun-Passives:RESISTOR0805-RES -> resistor:R-US_R0603
- R4: value 40.2K -> 330; device resistor:R-US_R0603 -> SparkFun-Passives:RESISTOR0805-RES
- R5: value 1K -> 330; device resistor:R-US_R0603 -> SparkFun-Passives:RESISTOR0805-RES
- R6: value 4.7K -> 10K
- R7: value 40.2K -> 4.7K; device resistor:R-US_R0603 -> SparkFun-Passives:RESISTOR0805-RES
- R8, R9: value 330 -> 4.7K
- U2: value Tiny85-20-SMT -> TPA2005D1DGN; device SparkFun-DigitalIC:ATTINY45TINY85-20-SMT -> SparkFun-AnalogIC:TPA2005D1DGN
- renumbered AMP_O to JP13, FET to FET1, FMIC_IO to JP1, FM_AOUT to JP12, GND to JP9, GND29 to JP11, GND31 to JP8, GND33 to JP10, LID to JP7, PWRIN to JP4, R15 to R12, SCLK_BUS to JP3, SDIO_BUS to JP2, STA_CH to SW1, U$1 to JP5, U$2 to JP6
Connections:
- net !RST: now also R2.2; no longer R9.2
- net !RST-L: now also R2.1, R6.2; no longer R10.2, R9.1
- net !SEN: now also R3.2; no longer R8.2
- net !SEN-L: now also R3.1, R9.1; no longer R14.1, R8.1
- net 3.3V: now also R7.2, R8.2, R9.2; no longer R13.2, R14.2, R6.2
- net A_IN: now also C9.2, R1.SIGNAL; no longer C14.2, U$5.SIGNAL
- net A_OUT: now also C13.1, R1.WIPER; no longer C9.1, U$5.WIPER
- net GND: now also C1.-, C10.2, C11.2, C12.2, C14.2, C18.1, C19.1, C20.1, C5.2, J2.6, R1.GND, R6.1, U2.GND@1, U2.GND@2, U3.GND; no longer AMP.GND@1, AMP.GND@2, C1.2, C11.1, C12.1, C13.2, C18.2, C19.-, C20.2, C3.2, C5.1, J1.6, R10.1, U$5.GND, U2.GND
- net LOUT: now also C9.1; no longer C14.1
- net N$1: now also C4.1; no longer C15.1
- net N$11: now also U3.PB3(ADC3); no longer U2.PB3(ADC3)
- net N$12: now also R14.2, U3.PB4(ADC2); no longer R5.2, U2.PB4(ADC2)
- net N$14: now also J1.ANT; no longer ANT.ANT
- net N$15: now also R1.SW_OUT; no longer U$5.SW_OUT
- net N$17: now also C2.1, C3.1; no longer C10.1, C8.1
- net N$18: now also C18.2, C19.2, C20.2, L3.2, U2.VDD; no longer AMP.VDD, C12.2, C16.2, C5.2, L4.2
- net N$2: now also C5.1; no longer C7.1
- net N$20: now also C15.1, U2.SHUTDOWN; no longer AMP.SHUTDOWN, C18.1
- net N$23: now also C16.2, R13.1; no longer C11.2, R4.1
- net N$3: now also C13.2, R11.1; no longer C9.2, R7.1
- net N$34: now also R1.SW_IN; no longer U$5.SW_IN
- net N$35: now also C6.1, R10.1; no longer C20.1, R1.1
- net N$4: now also R11.2, U2.IN+; no longer AMP.IN+, R7.2
- net N$5: now also R13.2, U2.IN-; no longer AMP.IN-, R4.2
- net N$6: now also C3.2; no longer C10.2
- net N$7: now also R14.1; no longer R5.1
- net N$8: now also R10.2; no longer R1.2
- net N$9: now also C10.1, C11.1, C7.1, C8.1, L2.2; no longer C1.1, C13.1, C2.1, C6.1, L3.2
- net OUT+: now also U2.OUT+; no longer AMP.OUT+
- net OUT-: now also U2.OUT-; no longer AMP.OUT-
- net PB1: now also J2.1, U3.PB1(MISO); no longer J1.1, U2.PB1(MISO)
- net PB5: now also J2.5, U3.PB5(NRES); no longer J1.5, U2.PB5(NRES)
- net SCLK: now also J2.3, R4.2, U3.PB2(SCK/ADC1); no longer J1.3, R3.2, U2.PB2(SCK/ADC1)
- net SCLK-L: now also R4.1, R8.1; no longer R3.1, R6.1
- net SDIO: now also J2.4, R5.2, U3.PB0(MOSI); no longer J1.4, R2.2, U2.PB0(MOSI)
- net SDIO-L: now also R5.1, R7.1; no longer R13.1, R2.1
- net VCC: now also C1.+, C12.1, C14.1, J2.2, L2.1, U3.VCC; no longer C19.+, C3.1, C4.1, J1.2, L4.1, U2.VCC
Other:
- moved on the sheet: C10, C11, C12, C13, C14, C15, C16, C17, C18, C2, C20, C3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

Commit message: Updated Sch & Layout
Began layout on the test board
Parts:
- added U$3: CE32A_DAYTON_SPKR, PR_Libraries:CE32A_DAYTON_SPKR
Connections:
- net OUT+: now also U$3.-
- net OUT-: now also U$3.+
Changed lines of the file:
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@@
 <setting verticaltext="up"/>
 </settings>
-<grid distance="0.1" unitdist="inch" unit="inch" style="lines" multiple="1" display="no" altdistance="0.01" altunitdist="inch" altunit="inch"/>
+<grid distance="0.01" unitdist="inch" unit="inch" style="lines" multiple="1" display="no" altdistance="0.01" altunitdist="inch" altunit="inch"/>
 <layers>
 <layer number="1" name="Top" color="4" fill="1" visible="no" active="no"/>
@@
 <part name="JP6" library="PR_Libraries" deviceset="BK-92_MPD_AA_BATT_CLIP" device=""/>
 <part name="GND10" library="SparkFun-Aesthetics" deviceset="GND" device=""/>
+<part name="U$3" library="PR_Libraries" deviceset="CE32A_DAYTON_SPKR" device=""/>
 </parts>
 <sheets>
@@
 <instance part="JP6" gate="BATT" x="25.4" y="104.14" rot="R180"/>
 <instance part="GND10" gate="1" x="33.02" y="96.266"/>
+<instance part="U$3" gate="G$1" x="228.346" y="25.146" rot="MR180"/>
 </instances>
 <busses>
@@
 <segment>
 <pinref part="U2" gate="G$1" pin="OUT-"/>
-<wire x1="192.024" y1="39.624" x2="223.266" y2="39.624" width="0.1524" layer="91"/>
+<wire x1="192.024" y1="39.624" x2="220.218" y2="39.624" width="0.1524" layer="91"/>
 <pinref part="JP13" gate="G$1" pin="2"/>
 <label x="224.028" y="39.116" size="2.1844" layer="95" rot="R180"/>
+<wire x1="220.218" y1="39.624" x2="223.266" y2="39.624" width="0.1524" layer="91"/>
+<wire x1="220.218" y1="39.624" x2="220.218" y2="22.606" width="0.1524" layer="91"/>
+<junction x="220.218" y="39.624"/>
+<pinref part="U$3" gate="G$1" pin="+"/>
+<wire x1="225.806" y1="22.606" x2="220.218" y2="22.606" width="0.1524" layer="91"/>
 </segment>
 </net>
@@
 <segment>
 <pinref part="U2" gate="G$1" pin="OUT+"/>
-<wire x1="192.024" y1="42.164" x2="223.266" y2="42.164" width="0.1524" layer="91"/>
+<wire x1="192.024" y1="42.164" x2="222.504" y2="42.164" width="0.1524" layer="91"/>
 <pinref part="JP13" gate="G$1" pin="1"/>
 <label x="224.028" y="44.45" size="2.1844" layer="95" rot="R180"/>
-</segment>
-</net>
+<wire x1="223.266" y1="42.164" x2="222.504" y2="42.164" width="0.1524" layer="91"/>
+<wire x1="222.504" y1="42.164" x2="222.504" y2="27.686" width="0.1524" layer="91"/>
+<wire x1="222.504" y1="27.686" x2="225.806" y2="27.686" width="0.1524" layer="91"/>
+<pinref part="U$3" gate="G$1" pin="-"/>
+<junction x="222.504" y="42.164"/>
+</segment>
+</net>
