File: EAGLE_CAD/PR9015.sch (EAGLE design)
At the start: 73 parts, among them J1 M3_SCREW_POST, SW1 C&K_PTS645

Commit message: Updated Lib / SCH / Layout
Added a resistor 0402 worthington footprint.
Todo:
-make the same for inductors
-clean up resistor 0402 traces
Parts:
- R11, R12, R13, R14, R15, R2, R4, R5, R7, R8, R9: device resistor:R-US_R0402 -> PR_Parts_Library:RES_SMT
Changed lines of the file:
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@@
 <part name="AMP" library="PR_Parts_Library" deviceset="TPA2005D1" device="DGN"/>
 <part name="GND27" library="SparkFun-Aesthetics" deviceset="GND" device=""/>
-<part name="R11" library="resistor" deviceset="R-US_" device="R0402" value="40.2K"/>
-<part name="R13" library="resistor" deviceset="R-US_" device="R0402" value="40.2K"/>
+<part name="R11" library="PR_Parts_Library" deviceset="RES_SMT" device="" value="40.2K"/>
+<part name="R13" library="PR_Parts_Library" deviceset="RES_SMT" device="" value="40.2K"/>
 <part name="C13" library="PR_Parts_Library" deviceset="CAP_SMT" device="" value=".033uf"/>
 <part name="C16" library="PR_Parts_Library" deviceset="CAP_SMT" device="" value=".033uf"/>
@@
 <part name="GND29" library="SparkFun-Aesthetics" deviceset="GND" device=""/>
 <part name="GND4" library="SparkFun-Aesthetics" deviceset="GND" device=""/>
-<part name="R12" library="resistor" deviceset="R-US_" device="R0402" value="10K"/>
+<part name="R12" library="PR_Parts_Library" deviceset="RES_SMT" device="" value="10K"/>
 <part name="GND24" library="SparkFun-Aesthetics" deviceset="GND" device=""/>
 <part name="P+1" library="supply1" deviceset="VCC" device=""/>
@@
 <part name="SUPPLY9" library="SparkFun-Aesthetics" deviceset="VCC" device=""/>
 <part name="GND32" library="SparkFun" deviceset="GND" device=""/>
-<part name="R14" library="resistor" deviceset="R-US_" device="R0402" value="1K"/>
+<part name="R14" library="PR_Parts_Library" deviceset="RES_SMT" device="" value="1K"/>
 <part name="GND6" library="SparkFun-Aesthetics" deviceset="GND" device=""/>
 <part name="L1" library="SparkFun-Passives" deviceset="INDUCTOR" device="0805" value="180nH"/>
@@
 <part name="FB2" library="SparkFun-Passives" deviceset="INDUCTOR" device="0805"/>
 <part name="FB3" library="SparkFun-Passives" deviceset="INDUCTOR" device="0805"/>
-<part name="R15" library="resistor" deviceset="R-US_" device="R0402" value="10K"/>
+<part name="R15" library="PR_Parts_Library" deviceset="RES_SMT" device="" value="10K"/>
 <part name="SUPPLY1" library="SparkFun-Aesthetics" deviceset="VCC" device=""/>
 <part name="JST_CONN" library="adafruit" deviceset="JST_2PIN" device="-SMT-RA"/>
@@
 <part name="C7" library="PR_Parts_Library" deviceset="CAP_SMT" device="" value="22n"/>
 <part name="C8" library="PR_Parts_Library" deviceset="CAP_SMT" device="" value=".1u"/>
-<part name="R2" library="resistor" deviceset="R-US_" device="R0402" value="330"/>
-<part name="R4" library="resistor" deviceset="R-US_" device="R0402" value="330"/>
-<part name="R5" library="resistor" deviceset="R-US_" device="R0402" value="330"/>
-<part name="R8" library="resistor" deviceset="R-US_" device="R0402" value="4.7k"/>
-<part name="R9" library="resistor" deviceset="R-US_" device="R0402" value="4.7k"/>
-<part name="R7" library="resistor" deviceset="R-US_" device="R0402" value="4.7k"/>
+<part name="R2" library="PR_Parts_Library" deviceset="RES_SMT" device="" value="330"/>
+<part name="R4" library="PR_Parts_Library" deviceset="RES_SMT" device="" value="330"/>
+<part name="R5" library="PR_Parts_Library" deviceset="RES_SMT" device="" value="330"/>
+<part name="R8" library="PR_Parts_Library" deviceset="RES_SMT" device="" value="4.7k"/>
+<part name="R9" library="PR_Parts_Library" deviceset="RES_SMT" device="" value="4.7k"/>
+<part name="R7" library="PR_Parts_Library" deviceset="RES_SMT" device="" value="4.7k"/>
 <part name="R6" library="resistor" deviceset="R-US_" device="R0402" value="10k"/>
 <part name="C10" library="PR_Parts_Library" deviceset="CAP_SMT" device="" value="22n"/>
@@
 <instance part="GND20" gate="1" x="91.44" y="66.04" rot="R90"/>
 <instance part="GND9" gate="1" x="27.94" y="15.24"/>
-<instance part="SUPPLY5" gate="1" x="10.16" y="73.66"/>
+<instance part="SUPPLY5" gate="G$1" x="10.16" y="73.66"/>
 <instance part="AMP" gate="G$1" x="172.72" y="40.64"/>
 <instance part="GND27" gate="1" x="167.64" y="22.86"/>
@@
 <instance part="GND3" gate="1" x="-27.94" y="129.54"/>
 <instance part="MCU" gate="G$1" x="175.26" y="124.46"/>
-<instance part="SUPPLY8" gate="1" x="154.94" y="132.08"/>
+<instance part="SUPPLY8" gate="G$1" x="154.94" y="132.08"/>
 <instance part="GND25" gate="1" x="154.94" y="116.84"/>
 <instance part="GND23" gate="1" x="139.7" y="121.92"/>
 <instance part="GND22" gate="1" x="129.54" y="121.92"/>
-<instance part="SUPPLY6" gate="1" x="129.54" y="139.7"/>
-<instance part="SUPPLY7" gate="1" x="139.7" y="139.7"/>
+<instance part="SUPPLY6" gate="G$1" x="129.54" y="139.7"/>
+<instance part="SUPPLY7" gate="G$1" x="139.7" y="139.7"/>
 <instance part="GND31" gate="1" x="226.06" y="106.68"/>
 <instance part="ISP" gate="G$1" x="220.98" y="127"/>
 <instance part="LED1" gate="G$1" x="205.74" y="101.6"/>
 <instance part="GND30" gate="1" x="205.74" y="91.44"/>
-<instance part="SUPPLY9" gate="1" x="231.14" y="137.16"/>
+<instance part="SUPPLY9" gate="G$1" x="231.14" y="137.16"/>
 <instance part="GND32" gate="1" x="231.14" y="116.84"/>
 <instance part="R14" gate="G$1" x="198.12" y="104.14" smashed="yes" rot="R180">
@@
 <attribute name="VALUE" x="205.994" y="123.952" size="1.778" layer="96" rot="R90"/>
 </instance>
-<instance part="SUPPLY1" gate="1" x="200.66" y="139.7"/>
+<instance part="SUPPLY1" gate="G$1" x="200.66" y="139.7"/>
 <instance part="JST_CONN" gate="G$1" x="220.98" y="38.1"/>
 <instance part="C2" gate="G$1" x="7.62" y="30.48"/>
@@
 <segment>
 <pinref part="MCU" gate="G$1" pin="VCC"/>
-<pinref part="SUPPLY8" gate="1" pin="VCC"/>
+<pinref part="SUPPLY8" gate="G$1" pin="VCC"/>
 <wire x1="160.02" y1="132.08" x2="154.94" y2="132.08" width="0.1524" layer="91"/>
 </segment>
 <segment>
 <pinref part="L2" gate="G$1" pin="1"/>
-<pinref part="SUPPLY5" gate="1" pin="VCC"/>
+<pinref part="SUPPLY5" gate="G$1" pin="VCC"/>
 <wire x1="17.78" y1="73.66" x2="10.16" y2="73.66" width="0.1524" layer="91"/>
 </segment>
@@
 <pinref part="ISP" gate="G$1" pin="2"/>
 <wire x1="231.14" y1="137.16" x2="231.14" y2="129.54" width="0.1524" layer="91"/>
-<pinref part="SUPPLY9" gate="1" pin="VCC"/>
-</segment>
-<segment>
-<pinref part="SUPPLY6" gate="1" pin="VCC"/>
+<pinref part="SUPPLY9" gate="G$1" pin="VCC"/>
+</segment>
+<segment>
+<pinref part="SUPPLY6" gate="G$1" pin="VCC"/>
 <pinref part="C12" gate="G$1" pin="1"/>
 <wire x1="129.54" y1="139.7" x2="129.54" y2="134.62" width="0.1524" layer="91"/>
 </segment>
 <segment>
-<pinref part="SUPPLY7" gate="1" pin="VCC"/>
+<pinref part="SUPPLY7" gate="G$1" pin="VCC"/>
 <wire x1="139.7" y1="139.7" x2="139.7" y2="137.16" width="0.1524" layer="91"/>
 <pinref part="C14" gate="G$1" pin="1"/>
@@
 <pinref part="R15" gate="G$1" pin="1"/>
 <wire x1="200.66" y1="132.08" x2="200.66" y2="139.7" width="0.1524" layer="91"/>
-<pinref part="SUPPLY1" gate="1" pin="VCC"/>
-</segment>
-<segment>
+<pinref part="SUPPLY1" gate="G$1" pin="VCC"/>
+</segment>
+<segment>
