File: EAGLE_CAD/PR9018.sch (EAGLE design)
At the start: 72 parts, among them SW1 C&K_PTS645, U1 SI4702-C19-GMR, X1 ABS25XTAL

Commit message: 9018 & PRTF01
9018 updated BOM and beginning layout & schematic of the PRXX test
fixture
Parts:
- C03, C23, C33: MFG_PN CL05B104KO5NNNC -> CL10B104KB8SFNC
Changed lines of the file:
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@@
 <?xml version="1.0" encoding="utf-8"?>
 <!DOCTYPE eagle SYSTEM "eagle.dtd">
-<eagle version="7.2.0">
+<eagle version="6.6.0">
 <drawing>
 <settings>
@@
 <part name="GND16" library="SparkFun" deviceset="GND" device=""/>
 <part name="C33" library="PR_Parts_Library" deviceset="C_SMT" device="_0603_CPL" value=".1uF">
-<attribute name="MFG_PN" value="CL05B104KO5NNNC"/>
+<attribute name="MFG_PN" value="CL10B104KB8SFNC"/>
 <attribute name="TOL" value="10%"/>
 <attribute name="VOLTAGE" value="16V"/>
 </part>
 <part name="C23" library="PR_Parts_Library" deviceset="C_SMT" device="_0603_CPL" value=".1uF">
-<attribute name="MFG_PN" value="CL05B104KO5NNNC"/>
+<attribute name="MFG_PN" value="CL10B104KB8SFNC"/>
 <attribute name="TOL" value="10%"/>
 <attribute name="VOLTAGE" value="16V"/>
@@
 </part>
 <part name="C03" library="PR_Parts_Library" deviceset="C_SMT" device="_0603_CPL" value=".1uF">
-<attribute name="MFG_PN" value="CL05B104KO5NNNC"/>
-<attribute name="TOL" value="10%"/>
-<attribute name="VOLTAGE" value="16V"/>
+<attribute name="MFG_PN" value="CL10B104KB8SFNC"/>
+<attribute name="TOL" value="10%"/>
+<attribute name="VOLTAGE" value="16V"/>

Commit message: changed JST to top
and fucked with tnames a bunch
Parts:
- R21, R22: MFG_PN RMCF0603FT12K0 -> RC0603FR-0712KL
- R23, R24: MFG_PN RMCF0603FT100K -> ERJ-3EKF1003V
- renumbered C01 to C1, C02 to C2, C03 to C3, C05 to C5, C08 to C8, JST_CONN to SPKR_PLUG, L01 to L1, R02 to R2, R03 to R3, R04 to R4, R05 to R5, R07 to R7, R08 to R8, TP1 to T1, TP10 to T10, TP11 to T11, TP12 to T12, TP13 to T13, TP14 to T14, TP15 to T15, TP16 to T16, TP17 to T17, TP2 to T2, TP3 to T3, TP4 to T4, TP5 to T5, TP6 to T6, TP7 to T7, TP8 to T8, TP9 to T9
