File: EAGLE_CAD/PR9019.brd (EAGLE design)
At the start: 70 x 70 mm, 73 parts

Commit message: pushed to pr9019, added production files
Parts:
- moved MARK3 0.41 mm to (67.0, 35.0)
Routing:
- net GND: vias 112 -> 118
Other:
- board text added: "PR9019 Born + tuned in Brooklyn http://thepublicrad.io"
- board text removed: "Brooklyn, NY By Centerline Labs"
