File: EAGLE_CAD/PR9019.sch (EAGLE design)
At the start: 72 parts, among them SW1 C&K_PTS645, U1 SI4702-C19-GMR, X1 ABS25XTAL

Commit message: pushed to pr9019, added production files
Parts:
- JP5, JP6: MFG_PN (none) -> 2 of BK92 - supplied by CL Labs
- R1: MFG_PN (none) -> RV170SF-43-20F-A10K - supplied by CL Labs
- U1: MFG_PN (none) -> Si4702 C19 GM - supplied by CL Labs
Other:
- note added: "PUBLIC RADIO PR9019 Production Board"
- note removed: "PUBLIC RADIO PR9017 Development Board"
Changed lines of the file:
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@@
 </classes>
 <parts>
-<part name="U1" library="PR_Parts_Library" deviceset="SI4702-C19-GMR" device="" value=""/>
+<part name="U1" library="PR_Parts_Library" deviceset="SI4702-C19-GMR" device="" value="">
+<attribute name="MFG_PN" value="Si4702 C19 GM - supplied by CL Labs"/>
+</part>
 <part name="GND13" library="SparkFun" deviceset="GND" device=""/>
 <part name="GND11" library="SparkFun" deviceset="GND" device=""/>
@@
 <part name="P+1" library="supply1" deviceset="VCC" device=""/>
 <part name="ANT_MOUNT" library="PR_Parts_Library" deviceset="M3_SCREW_POST" device="" value="DNP"/>
-<part name="R1" library="PR_Parts_Library" deviceset="RV170SF_TAIWANA_POT_SW" device="" value=""/>
+<part name="R1" library="PR_Parts_Library" deviceset="RV170SF_TAIWANA_POT_SW" device="" value="">
+<attribute name="MFG_PN" value="RV170SF-43-20F-A10K - supplied by CL Labs"/>
+</part>
 <part name="GND5" library="SparkFun-Aesthetics" deviceset="GND" device=""/>
 <part name="GND2" library="SparkFun-Aesthetics" deviceset="GND" device=""/>
@@
 <attribute name="MFG_PN" value="BAV99,215"/>
 </part>
-<part name="JP5" library="PR_Parts_Library" deviceset="BK-92_MPD_AA_BATT_CLIP" device="" value=""/>
-<part name="JP6" library="PR_Parts_Library" deviceset="BK-92_MPD_AA_BATT_CLIP" device="" value=""/>
+<part name="JP5" library="PR_Parts_Library" deviceset="BK-92_MPD_AA_BATT_CLIP" device="" value="">
+<attribute name="MFG_PN" value="2 of BK92 - supplied by CL Labs"/>
+</part>
+<part name="JP6" library="PR_Parts_Library" deviceset="BK-92_MPD_AA_BATT_CLIP" device="" value="">
+<attribute name="MFG_PN" value="2 of BK92 - supplied by CL Labs"/>
+</part>
 <part name="GND10" library="SparkFun-Aesthetics" deviceset="GND" device=""/>
 <part name="FB2" library="PR_Parts_Library" deviceset="L_SMT" device="_0805_ADAFRUIT">
@@
 <text x="157.48" y="144.78" size="2.54" layer="96">MCU
 ZONE 3x</text>
-<text x="-27.94" y="162.56" size="3.81" layer="96">PUBLIC RADIO PR9017
-Development Board </text>
+<text x="-27.94" y="162.56" size="3.81" layer="96">PUBLIC RADIO PR9019
+Production Board </text>
 <text x="22.098" y="109.474" size="2.54" layer="96">Fiducials </text>
 <text x="71.12" y="147.574" size="2.54" layer="96">Test Points </text>
