File: EAGLE_CAD/TestFixtures /PRTF02.sch (EAGLE design)
At the start: 40 parts

Commit message: PR9020 Gerbers
PR9020 Gerbers, organized folders
Parts:
- added U$20: PINHD-1X10, adafruit:PINHD-1X10
- added U1: V_REG_317SMD, SparkFun-PowerIC:V_REG_317SMD
Connections:
- new net N$1: U$19.TIP, U1.IN
- new net T1: U$2.P$1, U$20.1
- new net T2: U$20.2, U$3.P$1
- net GND: now also U$19.RING; no longer U$2.P$1, U$3.P$1
- net VCC: now also U1.OUT
Other:
- moved on the sheet: U$19
Changed lines of the file:
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@@
 <part name="U$19" library="adafruit" deviceset="2.1MMJACK" device="THM"/>
 <part name="ISP1" library="adafruit" deviceset="AVRISP" device="-6"/>
-<part name="GND2" library="SparkFun-Aesthetics" deviceset="GND" device=""/>
-<part name="GND3" library="SparkFun-Aesthetics" deviceset="GND" device=""/>
 <part name="GND4" library="SparkFun-Aesthetics" deviceset="GND" device=""/>
 <part name="P+1" library="supply1" deviceset="VCC" device=""/>
@@
 <part name="GND6" library="SparkFun-Aesthetics" deviceset="GND" device=""/>
 <part name="P+5" library="supply1" deviceset="VCC" device=""/>
+<part name="U1" library="SparkFun-PowerIC" deviceset="V_REG_317" device="SMD"/>
+<part name="GND7" library="SparkFun-Aesthetics" deviceset="GND" device=""/>
+<part name="P+6" library="supply1" deviceset="VCC" device=""/>
+<part name="U$20" library="adafruit" deviceset="PINHD-1X10" device=""/>
 </parts>
 <sheets>
@@
 <instance part="U$17" gate="G$1" x="147.32" y="78.74"/>
 <instance part="U$18" gate="G$1" x="160.02" y="78.74"/>
-<instance part="U$19" gate="G$1" x="256.54" y="144.78"/>
+<instance part="U$19" gate="G$1" x="256.54" y="147.32"/>
 <instance part="ISP1" gate="G$1" x="218.44" y="144.78"/>
-<instance part="GND2" gate="1" x="121.92" y="139.7"/>
-<instance part="GND3" gate="1" x="134.62" y="139.7"/>
 <instance part="GND4" gate="1" x="147.32" y="139.7"/>
 <instance part="P+1" gate="VCC" x="160.02" y="137.16" rot="R180"/>
@@
 <instance part="GND6" gate="1" x="236.22" y="139.7"/>
 <instance part="P+5" gate="VCC" x="238.76" y="147.32" rot="R270"/>
+<instance part="U1" gate="G$1" x="274.32" y="149.86"/>
+<instance part="GND7" gate="1" x="261.62" y="139.7"/>
+<instance part="P+6" gate="VCC" x="287.02" y="149.86" rot="R270"/>
+<instance part="U$20" gate="G$1" x="218.44" y="111.76"/>
 </instances>
 <busses>
@@
 </segment>
 <segment>
-<pinref part="U$2" gate="G$1" pin="P$1"/>
-<pinref part="GND2" gate="1" pin="GND"/>
-</segment>
-<segment>
-<pinref part="U$3" gate="G$1" pin="P$1"/>
-<pinref part="GND3" gate="1" pin="GND"/>
-</segment>
-<segment>
 <pinref part="U$4" gate="G$1" pin="P$1"/>
 <pinref part="GND4" gate="1" pin="GND"/>
@@
 <pinref part="GND6" gate="1" pin="GND"/>
 </segment>
+<segment>
+<pinref part="U$19" gate="G$1" pin="RING"/>
+<pinref part="GND7" gate="1" pin="GND"/>
+<wire x1="261.62" y1="142.24" x2="261.62" y2="144.78" width="0.1524" layer="91"/>
+</segment>
 </net>
 <net name="!RST" class="0">
@@
 <pinref part="P+5" gate="VCC" pin="VCC"/>
 </segment>
+<segment>
+<pinref part="U1" gate="G$1" pin="OUT"/>
+<pinref part="P+6" gate="VCC" pin="VCC"/>
+<wire x1="284.48" y1="149.86" x2="281.94" y2="149.86" width="0.1524" layer="91"/>
+</segment>
 </net>
 <net name="A_OUT" class="0">
@@
 </segment>
 </net>
+<net name="N$1" class="0">
+<segment>
+<pinref part="U$19" gate="G$1" pin="TIP"/>
+<pinref part="U1" gate="G$1" pin="IN"/>
+<wire x1="266.7" y1="149.86" x2="261.62" y2="149.86" width="0.1524" layer="91"/>
+</segment>
+</net>
+<net name="T2" class="0">
+<segment>
+<pinref part="U$3" gate="G$1" pin="P$1"/>
+<wire x1="134.62" y1="142.24" x2="134.62" y2="139.7" width="0.1524" layer="91"/>
+<label x="129.54" y="139.7" size="1.778" layer="95"/>
+</segment>
+<segment>
+<pinref part="U$20" gate="G$1" pin="2"/>
+<wire x1="215.9" y1="119.38" x2="208.28" y2="119.38" width="0.1524" layer="91"/>
+<label x="205.74" y="119.38" size="1.778" layer="95"/>
+</segment>
+</net>
+<net name="T1" class="0">
+<segment>
+<pinref part="U$2" gate="G$1" pin="P$1"/>
+<wire x1="121.92" y1="142.24" x2="121.92" y2="139.7" width="0.1524" layer="91"/>
+<label x="116.84" y="139.7" size="1.778" layer="95"/>
+</segment>
+<segment>
+<pinref part="U$20" gate="G$1" pin="1"/>
+<wire x1="215.9" y1="121.92" x2="208.28" y2="121.92" width="0.1524" layer="91"/>
+<label x="205.74" y="121.92" size="1.778" layer="95"/>
+</segment>
+</net>

Commit message: Test fixture updates
Initial schematic of the test fixture for PR9020.  No real layout done.
Parts:
- removed MARK1, MARK2, MARK3: FIDUCIAL, PR_Parts_Library:FIDUCIAL
- removed T1, T10, T11, T12, T13, T14, T15, T16, T17, T2, T3, T4, T5, T6, T7, T8, T9: (no value), PR_Parts_Library:TPTP20R
- removed U$20: PINHD-1X10, adafruit:PINHD-1X10
- added CN1: (no value), PR_Parts_Library:JST_2PIN-SMT-RA
- added J1: M3_SCREW_POST, PR_Parts_Library:M3_SCREW_POST
- added JP1, JP2: SMT/THJumper, SparkFun-Connectors:M02LOCK_LONGPADS
- added LED1: (no value), adafruit:LED5MM
- added R2: 1k, PR_Parts_Library:R_SMT_0805_ADAFRUIT
- added TO_MCU: PINHD-1X10, adafruit:PINHD-1X10
- added U$21: 0908MILL_MAX_SPRINGPIN, PR_Parts_Library:0908MILL_MAX_SPRINGPIN
Connections:
- removed net !RST: T10.TP
- removed net A_IN: R1.SIGNAL, T16.TP, U$17.P$1
- removed net SCLK: T11.TP
- removed net SDIO: T13.TP
- removed net SW: T8.TP, U$9.P$1
- removed net T1: U$2.P$1, U$20.1
- removed net T2: U$20.2, U$3.P$1
- new net ANT: J1.ANT, U$21.P$1
- new net DUTPRES: TO_MCU.1, U$2.P$1
- new net N$2: LED1.A, R2.2
- new net N$5: JP2.1, R1.SIGNAL
- new net N$6: JP1.2, R1.WIPER
- new net N$7: JP2.2, U$17.P$1
- new net TSW: TO_MCU.4, U$9.P$1
- net A_OUT: now also JP1.1; no longer R1.WIPER, T17.TP
- net GND: now also LED1.C, U$3.P$1; no longer T1.TP, T2.TP, T3.TP
- net LED/PB4: now also R2.1; no longer T9.TP
- net RESET: no longer T12.TP
- net SPK_OUT+: now also CN1.2; no longer T6.TP
- net SPK_OUT-: now also CN1.1; no longer T7.TP
- net SW_IN: now also TO_MCU.2; no longer R1.SW_IN, T14.TP
- net SW_OUT: now also TO_MCU.3; no longer R1.SW_OUT, T15.TP
- net VCC: no longer T4.TP, T5.TP
Other:
- note added: "Antenna"
- note added: "Ext Speaker"
- note added: "ISP"
- note added: "LED"
- note added: "MCU Connect"
- note added: "NOTES: - PSU, connects via dc barrel jack to a 3.3 vreg. -MCU header connects to tactile switch; device present (ground pad), and the two poles of the switched potentiometer (when populated). -LED, connects to an external led on the test fixture. -Ext Speaker, connects to JST jack on the fixture. -Switched Pot, allows for volume control when testing SMT only boards. Uses shunt jumpers when fully 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"
- note added: "POWER / GND"
- note added: "PR9020 Test Fixture"
- note added: "PSU / VReg"
- note added: "Switched Pot"
- note removed: "Fiducials"
- note removed: "MISO"
- note removed: "MOSI"
- note removed: "PUBLIC RADIO PR9020 Production Board"
- note removed: "RESET"
- note removed: "SCK"
- note removed: "Switch / Power"
- note removed: "Test Points"
- note removed: "ZONE 4x"
- moved on the sheet: ISP1, U$19, U1
