File: EAGLE_CAD/PR9021/PR9021.sch (EAGLE design)
At the start: 72 parts, among them SW1 C&K_PTS645, U1 SI4702-C19-GMR, X1 ABS25XTAL

Commit message: moved some stuff around, ran the xy script
Parts:
- R40: value DNP -> (none)
Changed lines of the file:
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@@
 <attribute name="VOLTAGE" value="16V"/>
 </part>
-<part name="R40" library="PR_Parts_Library" deviceset="R_SMT" device="_R0603_CPL" value="DNP">
+<part name="R40" library="PR_Parts_Library" deviceset="R_SMT" device="_R0603_CPL">
 <attribute name="MFG_PN" value="ERJ-3GEY0R00V"/>
 </part>
