File: EAGLE_CAD/PR9026/PR9026.brd (EAGLE design)
At the start: 65.9 x 66 mm, 60 parts, among them SW1 C&K_PTS645

Commit message: changed to ATTiny25
Parts:
- SPKR_PLACE: value DNP -> (none)
Changed lines of the file:
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@@
 <?xml version="1.0" encoding="utf-8"?>
 <!DOCTYPE eagle SYSTEM "eagle.dtd">
-<eagle version="6.6.0">
+<eagle version="7.7.0">
 <drawing>
 <settings>
@@
 <setting verticaltext="up"/>
 </settings>
-<grid distance="0.025" unitdist="mm" unit="mm" style="lines" multiple="1" display="yes" altdistance="0.1" altunitdist="mm" altunit="mm"/>
+<grid distance="1" unitdist="mm" unit="mm" style="dots" multiple="1" display="yes" altdistance="0.1" altunitdist="mm" altunit="mm"/>
 <layers>
 <layer number="1" name="Top" color="4" fill="1" visible="yes" active="yes"/>
@@
 <pass name="Default">
 <param name="RoutingGrid" value="50mil"/>
+<param name="AutoGrid" value="1"/>
+<param name="Efforts" value="0"/>
+<param name="TopRouterVariant" value="1"/>
 <param name="tpViaShape" value="round"/>
 <param name="PrefDir.1" value="|"/>
@@
 <attribute name="MFG_PN" value="AO3435" x="62.9" y="21.5" size="1.778" layer="27" display="off"/>
 </element>
-<element name="SPKR_PLACE" library="PR_Parts_Library" package="PR2024_SPKR_PLACE(SMD)" value="DNP" x="35" y="35" locked="yes"/>
+<element name="SPKR_PLACE" library="PR_Parts_Library" package="PR2024_SPKR_PLACE(SMD)" value="" x="35" y="35" locked="yes"/>
 <element name="T14" library="PR_Parts_Library" package="TP20R" value="" x="62" y="30" smashed="yes" rot="MR0">
 <attribute name="NAME" x="62.3936" y="31.5416" size="0.6096" layer="26" font="vector" ratio="16" rot="MR0"/>
