File: EAGLE_CAD/PR9026/PR9026.sch (EAGLE design)
At the start: 59 parts, among them SW1 C&K_PTS645, U1 SI4702-C19-GMR, X1 ABS25XTAL

Commit message: changed to ATTiny25
Parts:
- SPKR_PLACE: value DNP -> PR2024_SPKR_SMD
Changed lines of the file:
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@@
 <?xml version="1.0" encoding="utf-8"?>
 <!DOCTYPE eagle SYSTEM "eagle.dtd">
-<eagle version="6.6.0">
+<eagle version="7.7.0">
 <drawing>
 <settings>
@@
 <attribute name="MFG_PN" value="AO3435"/>
 </part>
-<part name="SPKR_PLACE" library="PR_Parts_Library" deviceset="PR2024_SPKR_SMD" device="" value="DNP"/>
+<part name="SPKR_PLACE" library="PR_Parts_Library" deviceset="PR2024_SPKR_SMD" device="" value=""/>
 <part name="T14" library="PR_Parts_Library" deviceset="TP" device="TP20R"/>
 <part name="T15" library="PR_Parts_Library" deviceset="TP" device="TP20R"/>
